File: Falcon Micro Remote/SchV1/Board1.kicad_sch (KiCad schematic)
At the start: 44 parts, among them J41 Conn_01x02_Male, J51 Conn_01x03_Male, SW31 SW_Push, SW51 SW_Push, SW61 SW_Push, SW62 SW_Push, SW63 SW_Push, SW64 SW_Push, SW71 SW_Push, SW72 SW_Push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

Commit message: Modified some files, pushing to keep things up to date
Parts:
- C11, C12, C31, C41, C42, C51: footprint Capacitor_SMD:C_0201_0603Metric -> Capacitor_SMD:C_0603_1608Metric
Changed lines of the file:
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@@
       (effects (font (size 1.27 1.27)) (justify left))
     )
-    (property "Footprint" "Capacitor_SMD:C_0201_0603Metric" (id 2) (at 98.1202 88.9 0)
+    (property "Footprint" "Capacitor_SMD:C_0603_1608Metric" (id 2) (at 98.1202 88.9 0)
       (effects (font (size 1.27 1.27)) hide)
     )
@@
     (property "Reference" "C51" (id 0) (at 92.71 183.515 90))
     (property "Value" "1uF" (id 1) (at 92.71 186.055 90))
-    (property "Footprint" "Capacitor_SMD:C_0201_0603Metric" (id 2) (at 96.52 188.8998 0)
+    (property "Footprint" "Capacitor_SMD:C_0603_1608Metric" (id 2) (at 96.52 188.8998 0)
       (effects (font (size 1.27 1.27)) hide)
     )
@@
     (property "Reference" "C31" (id 0) (at 37.465 183.515 90))
     (property "Value" "1uF" (id 1) (at 37.465 186.055 90))
-    (property "Footprint" "Capacitor_SMD:C_0201_0603Metric" (id 2) (at 41.275 188.8998 0)
+    (property "Footprint" "Capacitor_SMD:C_0603_1608Metric" (id 2) (at 41.275 188.8998 0)
       (effects (font (size 1.27 1.27)) hide)
     )
@@
       (effects (font (size 1.27 1.27)) (justify left))
     )
-    (property "Footprint" "Capacitor_SMD:C_0201_0603Metric" (id 2) (at 85.4202 88.9 0)
+    (property "Footprint" "Capacitor_SMD:C_0603_1608Metric" (id 2) (at 85.4202 88.9 0)
       (effects (font (size 1.27 1.27)) hide)
     )
@@
       (effects (font (size 1.27 1.27)) (justify left))
     )
-    (property "Footprint" "Capacitor_SMD:C_0201_0603Metric" (id 2) (at 52.4002 45.72 0)
+    (property "Footprint" "Capacitor_SMD:C_0603_1608Metric" (id 2) (at 52.4002 45.72 0)
       (effects (font (size 1.27 1.27)) hide)
     )
@@
       (effects (font (size 1.27 1.27)) (justify left))
     )
-    (property "Footprint" "Capacitor_SMD:C_0201_0603Metric" (id 2) (at 30.1752 45.72 0)
+    (property "Footprint" "Capacitor_SMD:C_0603_1608Metric" (id 2) (at 30.1752 45.72 0)
       (effects (font (size 1.27 1.27)) hide)
     )
@@
   (symbol_instances
     (path "/ecdc66b9-63fa-4592-a848-cf2a8650161c"
-      (reference "C11") (unit 1) (value "10uF") (footprint "Capacitor_SMD:C_0201_0603Metric")
+      (reference "C11") (unit 1) (value "10uF") (footprint "Capacitor_SMD:C_0603_1608Metric")
     )
     (path "/d7283c91-7bb2-432f-8745-cfa50fa7b1e1"
-      (reference "C12") (unit 1) (value "10uF") (footprint "Capacitor_SMD:C_0201_0603Metric")
+      (reference "C12") (unit 1) (value "10uF") (footprint "Capacitor_SMD:C_0603_1608Metric")
     )
     (path "/4e4c102e-27f0-4b53-8fd4-bfba6e43ed80"
-      (reference "C31") (unit 1) (value "1uF") (footprint "Capacitor_SMD:C_0201_0603Metric")
+      (reference "C31") (unit 1) (value "1uF") (footprint "Capacitor_SMD:C_0603_1608Metric")
     )
     (path "/58d3dc2f-83c3-40bd-8149-a9ae527ba7f7"
-      (reference "C41") (unit 1) (value "10uF") (footprint "Capacitor_SMD:C_0201_0603Metric")
+      (reference "C41") (unit 1) (value "10uF") (footprint "Capacitor_SMD:C_0603_1608Metric")
     )
     (path "/0b6934fa-e0da-47d3-b234-fe32ab606f89"
-      (reference "C42") (unit 1) (value "0.1uF") (footprint "Capacitor_SMD:C_0201_0603Metric")
+      (reference "C42") (unit 1) (value "0.1uF") (footprint "Capacitor_SMD:C_0603_1608Metric")
     )
     (path "/15a2b364-ca9c-4160-8997-0fd81c16f0f3"
-      (reference "C51") (unit 1) (value "1uF") (footprint "Capacitor_SMD:C_0201_0603Metric")
+      (reference "C51") (unit 1) (value "1uF") (footprint "Capacitor_SMD:C_0603_1608Metric")
     )
     (path "/5251da4a-69d3-4bed-9f5a-6273a802e449"
